File: ELP2-Boost_PFSC.kicad_pcb (KiCad board)
At the start: 2 copper layers, 130 x 150 mm, 44 parts, among them J1 Screw_Terminal_01x03, J2 Screw_Terminal_01x03, Q1 12n50C3, U1 UCC38050

Commit message: Got all the blocks a lot closer and named the testpoints on the silkscreen
Parts:
- moved J2 34.3 mm to (109.2, 53.8), turned to 0 degrees
- moved C8 16.9 mm to (96.9, 58.2)
- moved D6 14.0 mm to (119.5, 66.7), turned to 0 degrees
- moved C1 12.9 mm to (139.9, 127.3), turned to 0 degrees
- moved R11 12.2 mm to (119.5, 130.8)
- moved C9 11.9 mm to (118.5, 124.4)
- moved R2 10.2 mm to (136.2, 139.0)
- moved TP3 9.56 mm to (135.8, 127.8)
- moved R3 5.83 mm to (140.3, 136.7), turned to 0 degrees
- moved C10 4.92 mm to (131.3, 124.7)
- moved Rs1 3.95 mm to (144.0, 91.5)
- moved C4 3.07 mm to (146.2, 119.2)
- moved C6 3.07 mm to (128.4, 118.9)
- moved D1 3.07 mm to (135.2, 132.5)
- moved HS1 3.07 mm to (135.2, 86.2)
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Connections:
- TR1 pad 1: /ZCD -> Earth
- TR1 pad 5: Earth -> /ZCD
Routing:
- net /Out+: track 73.3 -> 46.3 mm
- net /Vcc: track 79.1 -> 64.8 mm
- net /PFC/Mult_In: track 44.8 -> 32.0 mm
- net Earth: track 188.5 -> 201.1 mm
- net Net-(D5-+): track 73.9 -> 84.0 mm
- net Net-(D7-K): track 23.3 -> 15.1 mm
- net Net-(D6-A): track 67.2 -> 66.5 mm
Other:
- board text added: "CS"
- board text added: "Projeto Boost PFC Alunos: Emanuel Staub Araldi e Cícero Eduardo Dick Junior Disciplina: Eletrônica de Potência II Professor: Joabel Moia"
- board text added: "Vcc"
- board text added: "Vo_Sense"
- board text removed: "Mult In"
